Commit message: Updating models to use more sensible origin points

File: src/turtle_pi/urdf/turtle_pi.urdf (robot description, URDF)
Before this commit: robot turtle_pi, 3 links, 2 joints
Joints:
- joint left_wheel_joint: origin xyz=-0.004304 0.072475 0.032413 rpy=0 0 0 -> xyz=-0.050850 0.085775 -0.011100 rpy=0 0 0
- joint right_wheel_joint: origin xyz=0.097396 0.072475 0.032413 rpy=0 0 0 -> xyz=0.050850 0.085775 -0.011100 rpy=0 0 0

Commit message: Initial updates to include Gazebo simulation

File: src/turtle_pi/urdf/turtle_pi.urdf (robot description, URDF)
Before this commit: robot turtle_pi, 3 links, 2 joints
Links:
- link base_link: mass None -> 1; geometry collision box size=0.22 0.10 0.05; visual mesh filename=package://turtle_pi/urdf/meshes/turtle_pi_chassis.dae
- link left_wheel: mass None -> 1; geometry collision cylinder length=0.025 radius=0.035; visual mesh filename=package://turtle_pi/urdf/meshes/turtle_pi_wheel.dae
- link right_wheel: mass None -> 1; geometry collision cylinder length=0.025 radius=0.035; visual mesh filename=package://turtle_pi/urdf/meshes/turtle_pi_wheel.dae
