Commit message: Adding simplified collision mesh for body

File: src/turtle_pi_description/urdf/turtle_pi.urdf (robot description, URDF)
Before this commit: robot turtle_pi, 3 links, 2 joints
Links:
- link base_link: geometry collision mesh filename=package://turtle_pi_description/urdf/meshes/turtle_pi_chass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; visual mesh filename=package://turtle_pi_description/urdf/meshes/turtle_pi_chass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
- link left_wheel: geometry collision cylinder length=0.025 radius=0.035; visual mesh filename=package://turtle_pi_description/urdf/meshes/turtle_pi_wheel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
- link right_wheel: geometry collision cylinder length=0.025 radius=0.035; visual mesh filename=package://turtle_pi_description/urdf/meshes/turtle_pi_wheel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

Commit message: Further simplifying collision mesh, and calculating better Inertia Tensor

File: src/turtle_pi_description/urdf/turtle_pi.urdf (robot description, URDF)
Before this commit: robot turtle_pi, 3 links, 2 joints
Links:
- link left_wheel: mass 1 -> 0.1
- link right_wheel: mass 1 -> 0.1

Commit message: Initial implementation of gazebo simulation with diff_drive control - Robot showing up black for some reason??

File: src/turtle_pi_description/urdf/turtle_pi.urdf (robot description, URDF)
Before this commit: robot turtle_pi, 3 links, 2 joints
Joints:
- joint left_wheel_joint: axis 1 0 0 -> -1 0 0
- joint right_wheel_joint: axis 1 0 0 -> -1 0 0

Commit message: Adding camera simulation in gazebo, and bumping up max speed of robot

File: src/turtle_pi_description/urdf/turtle_pi.urdf (robot description, URDF)
Before this commit: robot turtle_pi, 3 links, 2 joints
Links:
- added link camera_link; visual box size=0.01 0.01 0.01
Joints:
- added joint camera_joint: type fixed, parent base_link, child camera_link, origin xyz=0 0.15 0.05 rpy=0 0 ${M_PI/2}

Commit message: Simulation mostly working

File: src/turtle_pi_description/urdf/turtle_pi.urdf (robot description, URDF)
Before this commit: robot turtle_pi, 4 links, 3 joints
Links:
- added link base_footprint
Joints:
- added joint base_joint: type fixed, parent base_footprint, child base_link, origin xyz=0 0 0.010 rpy=0 0 0

Commit message: Adding Kinect simulation instead of laser scanner.

File: src/turtle_pi_description/urdf/turtle_pi.urdf (robot description, URDF)
Before this commit: robot turtle_pi, 5 links, 4 joints
Links:
- added link camera_depth_link
Joints:
- added joint camera_depth_joint: type fixed, parent camera_link, child camera_depth_link, origin xyz=0 0 0 rpy=${-M_PI/2} 0 ${-M_PI/2} 
